File: Board Layouts/Main CPU Board/Buffers.sch (KiCad schematic (older format))
At the start: 8 parts, among them U10 74LS367, U11 74LS367, U12 74LS367, U13 74LS367, U14 74LS367, U7 74LS04, U8 74LS367, U9 74LS367

Commit message: Working on schematics and board layouts
Parts:
- renumbered U13 to U10, U14 to U11, U7 to U4, U8 to U5, U9 to U6, U10 to U7, U11 to U8, U12 to U9
Changed lines of the file:
@@
 $Descr A3 16535 11693
 encoding utf-8
-Sheet 2 2
+Sheet 2 3
 Title "Data and Address Buffers"
 Date "2019-03-23"
@@
 $EndDescr
 $Comp
-L 74xx:74LS367 U8
+L 74xx:74LS367 U5
 U 1 1 5CAC7860
 P 6500 4400
-F 0 "U8" H 6700 5050 50  0000 C CNN
+F 0 "U5" H 6700 5050 50  0000 C CNN
 F 1 "74LS367" H 6700 4950 50  0000 C CNN
 F 2 "" H 6500 4400 50  0001 C CNN
@@
 $EndComp
 $Comp
-L power:+5V #PWR014
+L power:+5V #PWR06
 U 1 1 5CACB1DD
 P 6500 3700
-F 0 "#PWR014" H 6500 3550 50  0001 C CNN
+F 0 "#PWR06" H 6500 3550 50  0001 C CNN
 F 1 "+5V" H 6515 3873 50  0000 C CNN
 F 2 "" H 6500 3700 50  0001 C CNN
@@
 $EndComp
 $Comp
-L power:GND #PWR015
+L power:GND #PWR07
 U 1 1 5CACB45F
 P 6500 5100
-F 0 "#PWR015" H 6500 4850 50  0001 C CNN
+F 0 "#PWR07" H 6500 4850 50  0001 C CNN
 F 1 "GND" H 6505 4927 50  0000 C CNN
 F 2 "" H 6500 5100 50  0001 C CNN
@@
 	6000 4700 6000 4800
 $Comp
-L 74xx:74LS367 U9
+L 74xx:74LS367 U6
 U 1 1 5CACD006
 P 6500 6250
-F 0 "U9" H 6700 6900 50  0000 C CNN
+F 0 "U6" H 6700 6900 50  0000 C CNN
 F 1 "74LS367" H 6700 6800 50  0000 C CNN
 F 2 "" H 6500 6250 50  0001 C CNN
@@
 $EndComp
 $Comp
-L power:+5V #PWR016
+L power:+5V #PWR08
 U 1 1 5CACD00C
 P 6500 5550
-F 0 "#PWR016" H 6500 5400 50  0001 C CNN
+F 0 "#PWR08" H 6500 5400 50  0001 C CNN
 F 1 "+5V" H 6515 5723 50  0000 C CNN
 F 2 "" H 6500 5550 50  0001 C CNN
@@
 $EndComp
 $Comp
-L power:GND #PWR017
+L power:GND #PWR09
 U 1 1 5CACD012
 P 6500 6950
-F 0 "#PWR017" H 6500 6700 50  0001 C CNN
+F 0 "#PWR09" H 6500 6700 50  0001 C CNN
 F 1 "GND" H 6505 6777 50  0000 C CNN
 F 2 "" H 6500 6950 50  0001 C CNN
@@
 	6000 6550 6000 6650
 $Comp
-L 74xx:74LS367 U10
+L 74xx:74LS367 U7
 U 1 1 5CACE81B
 P 6500 8100
-F 0 "U10" H 6700 8750 50  0000 C CNN
+F 0 "U7" H 6700 8750 50  0000 C CNN
 F 1 "74LS367" H 6700 8650 50  0000 C CNN
 F 2 "" H 6500 8100 50  0001 C CNN
@@
 $EndComp
 $Comp
-L power:+5V #PWR018
+L power:+5V #PWR010
 U 1 1 5CACE821
 P 6500 7400
-F 0 "#PWR018" H 6500 7250 50  0001 C CNN
+F 0 "#PWR010" H 6500 7250 50  0001 C CNN
 F 1 "+5V" H 6515 7573 50  0000 C CNN
 F 2 "" H 6500 7400 50  0001 C CNN
@@
 $EndComp
 $Comp
-L power:GND #PWR019
+L power:GND #PWR011
 U 1 1 5CACE827
 P 6500 8800
-F 0 "#PWR019" H 6500 8550 50  0001 C CNN
+F 0 "#PWR011" H 6500 8550 50  0001 C CNN
 F 1 "GND" H 6505 8627 50  0000 C CNN
 F 2 "" H 6500 8800 50  0001 C CNN
@@
 	6000 8400 6000 8500
 $Comp
-L 74xx:74LS367 U11
+L 74xx:74LS367 U8
 U 1 1 5CAD0672
 P 9850 3650
-F 0 "U11" H 10050 4300 50  0000 C CNN
+F 0 "U8" H 10050 4300 50  0000 C CNN
 F 1 "74LS367" H 10050 4200 50  0000 C CNN
 F 2 "" H 9850 3650 50  0001 C CNN
@@
 $EndComp
 $Comp
-L power:+5V #PWR020
+L power:+5V #PWR012
 U 1 1 5CAD0678
 P 9850 2950
-F 0 "#PWR020" H 9850 2800 50  0001 C CNN
+F 0 "#PWR012" H 9850 2800 50  0001 C CNN
 F 1 "+5V" H 9865 3123 50  0000 C CNN
 F 2 "" H 9850 2950 50  0001 C CNN
@@
 $EndComp
 $Comp
-L power:GND #PWR021
+L power:GND #PWR013
 U 1 1 5CAD067E
 P 9850 4350
-F 0 "#PWR021" H 9850 4100 50  0001 C CNN
+F 0 "#PWR013" H 9850 4100 50  0001 C CNN
 F 1 "GND" H 9855 4177 50  0000 C CNN
 F 2 "" H 9850 4350 50  0001 C CNN
@@
 $EndComp
 $Comp
-L 74xx:74LS367 U12
+L 74xx:74LS367 U9
 U 1 1 5CAD134A
 P 9850 5500
-F 0 "U12" H 10050 6150 50  0000 C CNN
+F 0 "U9" H 10050 6150 50  0000 C CNN
 F 1 "74LS367" H 10050 6050 50  0000 C CNN
 F 2 "" H 9850 5500 50  0001 C CNN
@@
 $EndComp
 $Comp
-L power:+5V #PWR022
+L power:+5V #PWR014
 U 1 1 5CAD1350
 P 9850 4800
-F 0 "#PWR022" H 9850 4650 50  0001 C CNN
+F 0 "#PWR014" H 9850 4650 50  0001 C CNN
 F 1 "+5V" H 9865 4973 50  0000 C CNN
 F 2 "" H 9850 4800 50  0001 C CNN
@@
 $EndComp
 $Comp
-L power:GND #PWR023
+L power:GND #PWR015
 U 1 1 5CAD1356
 P 9850 6200
-F 0 "#PWR023" H 9850 5950 50  0001 C CNN
+F 0 "#PWR015" H 9850 5950 50  0001 C CNN
 F 1 "GND" H 9855 6027 50  0000 C CNN
 F 2 "" H 9850 6200 50  0001 C CNN
@@
 $EndComp
 $Comp
-L 74xx:74LS367 U13
+L 74xx:74LS367 U10
 U 1 1 5CAD342E
 P 9850 7350
-F 0 "U13" H 10050 8000 50  0000 C CNN
+F 0 "U10" H 10050 8000 50  0000 C CNN
 F 1 "74LS367" H 10050 7900 50  0000 C CNN
 F 2 "" H 9850 7350 50  0001 C CNN
@@
 $EndComp
 $Comp
-L power:+5V #PWR024
+L power:+5V #PWR016
 U 1 1 5CAD3434
 P 9850 6650
-F 0 "#PWR024" H 9850 6500 50  0001 C CNN
+F 0 "#PWR016" H 9850 6500 50  0001 C CNN
 F 1 "+5V" H 9865 6823 50  0000 C CNN
 F 2 "" H 9850 6650 50  0001 C CNN
@@
 $EndComp
 $Comp
-L power:GND #PWR025
+L power:GND #PWR017
 U 1 1 5CAD343A
 P 9850 8050
-F 0 "#PWR025" H 9850 7800 50  0001 C CNN
+F 0 "#PWR017" H 9850 7800 50  0001 C CNN
 F 1 "GND" H 9855 7877 50  0000 C CNN
 F 2 "" H 9850 8050 50  0001 C CNN
@@
 $EndComp
 $Comp
-L 74xx:74LS367 U14
+L 74xx:74LS367 U11
 U 1 1 5CAD4FBD
 P 9850 9200
-F 0 "U14" H 10050 9850 50  0000 C CNN
+F 0 "U11" H 10050 9850 50  0000 C CNN
 F 1 "74LS367" H 10050 9750 50  0000 C CNN
 F 2 "" H 9850 9200 50  0001 C CNN
@@
 $EndComp
 $Comp
-L power:+5V #PWR026
+L power:+5V #PWR018
 U 1 1 5CAD4FC3
 P 9850 8500
-F 0 "#PWR026" H 9850 8350 50  0001 C CNN
+F 0 "#PWR018" H 9850 8350 50  0001 C CNN
 F 1 "+5V" H 9865 8673 50  0000 C CNN
 F 2 "" H 9850 8500 50  0001 C CNN
@@
 $EndComp
 $Comp
-L power:GND #PWR027
+L power:GND #PWR019
 U 1 1 5CAD4FC9
 P 9850 9900
-F 0 "#PWR027" H 9850 9650 50  0001 C CNN
+F 0 "#PWR019" H 9850 9650 50  0001 C CNN
 F 1 "GND" H 9855 9727 50  0000 C CNN
 F 2 "" H 9850 9900 50  0001 C CNN
@@
 Connection ~ 9200 5800
 $Comp
-L 74xx:74LS04 U7
+L 74xx:74LS04 U4
 U 3 1 5CB0577A
 P 10450 6550
-F 0 "U7" V 10350 6650 50  0000 R CNN
+F 0 "U4" V 10350 6650 50  0000 R CNN
 F 1 "74LS04" V 10495 6370 50  0001 R CNN
 F 2 "" H 10450 6550 50  0001 C CNN
@@
 	10450 9500 10350 9500
 $Comp
-L 74xx:74LS04 U7
+L 74xx:74LS04 U4
 U 2 1 5CB0FB49
 P 9200 2800
-F 0 "U7" V 9154 2980 50  0000 L CNN
+F 0 "U4" V 9154 2980 50  0000 L CNN
 F 1 "74LS04" V 9245 2980 50  0000 L CNN
 F 2 "" H 9200 2800 50  0001 C CNN
@@
 $EndComp
 $Comp
-L 74xx:74LS04 U7
+L 74xx:74LS04 U4
 U 1 1 5CB13ACE
 P 5600 3800
-F 0 "U7" H 5600 4117 50  0000 C CNN
+F 0 "U4" H 5600 4117 50  0000 C CNN
 F 1 "74LS04" H 5600 4026 50  0000 C CNN
 F 2 "" H 5600 3800 50  0001 C CNN
