File: Board Layouts/Main CPU Board/Main CPU Board.sch (KiCad schematic (older format))
At the start: 15 parts, among them SW1 SW_Push_SPDT, SW2 SW_SPDT, U1 74LS04, U2 74LS04, U3 74LS00, U4 Z80CPU, U5 74LS121, U6 74HC74, X1 1MHz

Commit message: Working on schematics and board layouts
Parts:
- removed C1: 1n, symbol Device:CP
- removed R1, R2, R4, R5: 4k7, symbol Device:R
- removed R3: 1k, symbol Device:R
- removed SW1: SW_Push_SPDT, symbol Switch:SW_Push_SPDT
- removed SW2: SW_SPDT, symbol Switch:SW_SPDT
- removed U3: 74LS00, symbol 74xx:74LS00
- removed U5: 74LS121, symbol 74xx:74LS121
- removed U6: 74HC74, symbol 74xx:74HC74
- renumbered U4 to U3
Connections:
- no-connect marks 8 -> 3
