File: Board Layouts/Front Panel/Front Panel.kicad_pcb (KiCad board)
At the start: 2 copper layers, 85 parts, among them J1 Conn_02x18_Odd_Even, SW1 SW_Push_SPDT, SW2 SW_Push, SW3 SW_Push, SW4 SW_SPDT, U1 74LS04, U10 74LS04, U2 74LS04, U3 74LS04, U4 7400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

Commit message: Working on board layouts and schematics
Parts:
- added C10: 10n, Capacitor_THT:C_Rect_L4.0mm_W2.5mm_P2.50mm, F.Cu at (229.9, 132.1)
- added C11: 10n, Capacitor_THT:C_Rect_L4.0mm_W2.5mm_P2.50mm, F.Cu at (210.8, 132.1)
- added C2: 10n, Capacitor_THT:C_Rect_L4.0mm_W2.5mm_P2.50mm, F.Cu at (99.1, 132.1)
- added C3: 10n, Capacitor_THT:C_Rect_L4.0mm_W2.5mm_P2.50mm, F.Cu at (59.6, 134.6)
- added C4: 10n, Capacitor_THT:C_Rect_L4.0mm_W2.5mm_P2.50mm, F.Cu at (27.9, 134.6)
- added C5: 10n, Capacitor_THT:C_Rect_L4.0mm_W2.5mm_P2.50mm, F.Cu at (262.9, 64.8)
- added C6: 10n, Capacitor_THT:C_Rect_L4.0mm_W2.5mm_P2.50mm, F.Cu at (242.5, 25.4)
- added C7: 10n, Capacitor_THT:C_Rect_L4.0mm_W2.5mm_P2.50mm, F.Cu at (280.7, 64.8)
- added C8: 10n, Capacitor_THT:C_Rect_L4.0mm_W2.5mm_P2.50mm, F.Cu at (162.6, 132.1)
- added C9: 10n, Capacitor_THT:C_Rect_L4.0mm_W2.5mm_P2.50mm, F.Cu at (144.8, 132.1)
Connections:
- U1 pad 14: (no net) -> +5V
- U1 pad 7: (no net) -> GND
- U10 pad 14: (no net) -> +5V
- U10 pad 7: (no net) -> GND
- U2 pad 14: (no net) -> +5V
- U2 pad 7: (no net) -> GND
- U3 pad 14: (no net) -> +5V
- U3 pad 7: (no net) -> GND
- U4 pad 14: (no net) -> +5V
- U4 pad 7: (no net) -> GND
- U6 pad 14: (no net) -> +5V
- U6 pad 7: (no net) -> GND
- U7 pad 14: (no net) -> +5V
- U7 pad 7: (no net) -> GND
- U8 pad 14: (no net) -> +5V
- U8 pad 7: (no net) -> GND
- U9 pad 14: (no net) -> +5V
- U9 pad 7: (no net) -> GND
Routing:
- net Net-(C1-Pad1): track 0.00 -> 9.94 mm
- net +5V: track 215.9 -> 224.8 mm
- net Net-(C1-Pad2): track 0.00 -> 3.83 mm
