File: Board Layouts/Front Panel/Front Panel.sch (KiCad schematic (older format))
At the start: 85 parts, among them J1 Conn_02x18_Odd_Even, SW1 SW_Push_SPDT, SW2 SW_Push, SW3 SW_Push, SW4 SW_SPDT, U1 74LS04, U10 74LS04, U2 74LS04, U3 74LS04, U4 7400, U5 74LS121, U6 74LS74, U7 74LS04, U8 74LS04, U9 74LS04

Commit message: Working on board layouts and schematics
Parts:
- added C10, C11, C2, C3, C4, C5, C6, C7, C8, C9: 10n, Capacitor_THT:C_Rect_L4.0mm_W2.5mm_P2.50mm, symbol Device:C
- added unit 7 of U1
- added unit 7 of U10
- added unit 7 of U2
- added unit 7 of U3
- added unit 5 of U4
- added unit 3 of U6
- added unit 7 of U7
- added unit 7 of U8
- added unit 7 of U9
Connections:
- net +5V: now also C10.1, C11.1, C2.1, C3.1, C4.1, C5.1, C6.1, C7.1, C8.1, C9.1, U1.14 (VCC), U10.14 (VCC), U2.14 (VCC), U3.14 (VCC), U4.14 (VCC), U6.14 (VCC), U7.14 (VCC), U8.14 (VCC), U9.14 (VCC)
- net GND: now also C10.2, C11.2, C2.2, C3.2, C4.2, C5.2, C6.2, C7.2, C8.2, C9.2, U1.7 (GND), U10.7 (GND), U2.7 (GND), U3.7 (GND), U4.7 (GND), U6.7 (GND), U7.7 (GND), U8.7 (GND), U9.7 (GND)

Commit message: Working on schematics
Changed lines of the file:
@@
 EESchema Schematic File Version 4
+LIBS:Front Panel-cache
 EELAYER 29 0
 EELAYER END
 $Descr A3 16535 11693
 encoding utf-8
-Sheet 1 1
+Sheet 1 2
 Title "Front Panel"
 Date "2019-03-23"
@@
 	1    0    0    -1
 $EndComp
+$Sheet
+S 6750 4850 550  500
+U 5C99B4A2
+F0 "Hex to 7-Segment Decoder" 50
+F1 "Hex to 7-Segment Decoder.sch" 50
+F2 "A0" I L 6750 4950 50
+F3 "A1" I L 6750 5050 50
+F4 "A2" I L 6750 5150 50
+F5 "A3" I L 6750 5250 50
+$EndSheet
 $EndSCHEMATC
