File: Board Layouts/Printer Driver/Printer Driver.kicad_pcb (KiCad board)
At the start: 2 copper layers, 25 parts, among them J1 USB_B, J2 Conn_01x06, J3 Conn_01x03, J4 8P8C, J5 DB25_Female_MountingHoles, U1 FT230XS, U2 PIC16F1503-IP, U3 74HC595, U4 PCA9615

Commit message: Routed pcb added bom for printer driver
Parts:
- added R10: 120, Resistor_THT:R_Axial_DIN0207_L6.3mm_D2.5mm_P10.16mm_Horizontal, F.Cu at (156.5, 76.2)
- added R11: 600, Resistor_THT:R_Axial_DIN0207_L6.3mm_D2.5mm_P10.16mm_Horizontal, F.Cu at (156.5, 89.2)
- added R12: 600, Resistor_THT:R_Axial_DIN0207_L6.3mm_D2.5mm_P10.16mm_Horizontal, F.Cu at (151.1, 62.5)
- added R13: 120, Resistor_THT:R_Axial_DIN0207_L6.3mm_D2.5mm_P10.16mm_Horizontal, F.Cu at (151.1, 76.2)
- added R14: 600, Resistor_THT:R_Axial_DIN0207_L6.3mm_D2.5mm_P10.16mm_Horizontal, F.Cu at (151.1, 89.2)
- added R7: 2k, Resistor_THT:R_Axial_DIN0207_L6.3mm_D2.5mm_P10.16mm_Horizontal, F.Cu at (115.8, 86.4)
- added R8: 2k, Resistor_THT:R_Axial_DIN0207_L6.3mm_D2.5mm_P10.16mm_Horizontal, F.Cu at (112.0, 88.9)
- added R9: 600, Resistor_THT:R_Axial_DIN0207_L6.3mm_D2.5mm_P10.16mm_Horizontal, F.Cu at (156.5, 62.4)
- added REF**: MountingHole_4.3mm_M4, MountingHole:MountingHole_4.3mm_M4, F.Cu at (53.3, 116.8)
- added REF**: MountingHole_4.3mm_M4, MountingHole:MountingHole_4.3mm_M4, F.Cu at (161.3, 116.8)
- added REF**: MountingHole_4.3mm_M4, MountingHole:MountingHole_4.3mm_M4, F.Cu at (161.3, 53.3)
- added REF**: MountingHole_4.3mm_M4, MountingHole:MountingHole_4.3mm_M4, F.Cu at (53.3, 53.3)
- moved J3 81.5 mm to (112.4, 117.9), turned to 0 degrees
- moved C4 66.9 mm to (114.9, 107.7), turned to 0 degrees
- moved J2 61.2 mm to (112.4, 71.1)
- moved C6 48.3 mm to (102.4, 72.4)
- moved U2 48.3 mm to (99.8, 76.2)
- moved U4 17.9 mm to (142.7, 82.0)
- moved C7 12.0 mm to (87.6, 78.7), turned to 270 degrees
- moved C8 8.83 mm to (141.2, 77.2)
- renumbered J5 to J4, J4 to J5
Routing:
- net GND: track 0.00 -> 293.1 mm, vias 0 -> 2
- net +5V: track 0.00 -> 204.5 mm, vias 0 -> 2
- net Net-(R7-Pad1): track 0.00 -> 63.3 mm, vias 0 -> 1
- net Net-(R8-Pad1): track 0.00 -> 61.8 mm, vias 0 -> 2
- net Net-(J5-Pad1): track 0.00 -> 50.9 mm, vias 0 -> 1
- net Net-(J2-Pad4): track 0.00 -> 50.5 mm, vias 0 -> 1
- net Net-(U1-Pad6): track 0.00 -> 49.6 mm, vias 0 -> 3
- net Net-(U1-Pad2): track 0.00 -> 45.6 mm, vias 0 -> 3
- net Net-(J5-Pad7): track 0.00 -> 44.4 mm
- net Net-(J2-Pad5): track 0.00 -> 42.1 mm, vias 0 -> 2
- net Net-(U1-Pad4): track 0.00 -> 41.6 mm, vias 0 -> 2
- net Net-(C3-Pad1): track 0.00 -> 37.6 mm
- net Net-(J4-Pad9): track 0.00 -> 37.0 mm
- net Net-(J5-Pad2): track 0.00 -> 35.8 mm, vias 0 -> 2
- net Net-(J5-Pad8): track 0.00 -> 33.5 mm
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Other:
- board outline added: 118.1 x 73.7 mm
