File: Board Layouts/Printer Driver/Printer Driver.sch (KiCad schematic (older format))
At the start: 4 parts

Commit message: Working on schematics
Parts:
- added C? (x2): 47p, symbol Device:C
- added C?: 100v, symbol Device:C
- added D? (x2): LED, symbol Device:LED
- added J?: USB_B, symbol Connector:USB_B
- added R?: 4k7, symbol Device:R
- added R?: 10k, symbol Device:R
- added R? (x2): 27, symbol Device:R
- added R? (x2): 270, symbol Device:R
- added U?: FT230XS, Package_SO:SSOP-16_3.9x4.9mm_P0.635mm, symbol Interface_USB:FT230XS
Connections:
- net +5V: now also C?.1, D?.2 (A), D?.2 (A), R?.1, R?.1, U?.10 (3V3OUT), U?.11 (~RESET), U?.12 (VCC), U?.3 (VCCIO), U?.8 (USBDP), U?.9 (USBDM)
- net GND: now also C?.2, C?.2, C?.2, J?.4 (GND), R?.2, U?.13 (GND), U?.5 (GND)
- new net: R?.2, U?.14 (CBUS1)
- new net: R?.1, R?.2, U?.16 (CBUS3)
- new net: R?.2, U?.7 (CBUS2)
- new net: J?.1 (VBUS), R?.1
- new net: C?.1, J?.2 (D-), R?.2
- new net: C?.1, J?.3 (D+), R?.2
- new net: D?.1 (K), R?.1 (x2)

Commit message: Working on schematics and board routing
Parts:
- added C4: 470u, Capacitor_THT:CP_Radial_D8.0mm_P3.50mm, symbol Device:CP
- added C5, C6, C7, C8: 10n, Capacitor_THT:C_Rect_L4.0mm_W2.5mm_P2.50mm, symbol Device:C
- added J3: Conn_01x03, Connector_JST:JST_VH_B3PS-VH_1x03_P3.96mm_Horizontal, symbol Connector_Generic:Conn_01x03
- added J4: 8P8C, Connector_RJ:RJ45_Amphenol_54602-x08_Horizontal, symbol Connector:8P8C
- added U4: PCA9615, Package_SO:TSSOP-10_3x3mm_P0.5mm, symbol Custom_Parts:PCA9615
- C1, C2: renamed from C?; footprint (none) -> Capacitor_THT:C_Rect_L4.0mm_W2.5mm_P2.50mm
- C3: renamed from C?; value 100v -> 100n; footprint (none) -> Capacitor_THT:C_Rect_L4.0mm_W2.5mm_P2.50mm
- D1, D2: renamed from D?; footprint (none) -> LED_THT:LED_D5.0mm
- J1: renamed from J?; footprint (none) -> Connector_USB:USB_B_OST_USB-B1HSxx_Horizontal
- J2: renamed from J?; footprint (none) -> Connector_PinHeader_2.54mm:PinHeader_1x06_P2.54mm_Vertical
- J5: renamed from J?; footprint (none) -> Connector_Dsub:DSUB-25_Female_Horizontal_P2.77x2.84mm_EdgePinOffset9.90mm_Housed_MountingHolesOffset11.32mm
- R1, R2, R3, R4, R5, R6: renamed from R?; footprint (none) -> Resistor_THT:R_Axial_DIN0207_L6.3mm_D2.5mm_P10.16mm_Horizontal
- U2: renamed from U?; footprint (none) -> Package_DIP:DIP-14_W7.62mm_Socket
- U3: renamed from U?; footprint (none) -> Package_DIP:DIP-16_W7.62mm
- gave numbers to parts that had none: 1
Connections:
- net +5V: now also U3.10 (~SRCLR), C4.1, C5.1, C6.1, C7.1, C8.1, J3.1 (Pin_1), U4.1 (Vdd(a)), U4.10 (Vdd(b)); no longer C3.1, D1.2 (A), D2.2 (A), R3.1, R4.1, U1.10 (3V3OUT), U1.11 (~RESET), U1.3 (VCCIO), U1.8 (USBDP), U1.9 (USBDM)
- net GND: now also U3.13 (~OE), C4.2, C5.2, C6.2, C7.2, C8.2, J3.3 (Pin_3), U4.5 (Vss); no longer J5.0 (PAD), U3.10 (~SRCLR)
- net at J5.1: now also J2.4 (Pin_4), U2.13 (RA0/AN0/DACOUT1/C1IN+/ICSPDAT); no longer U2.10 (SCK/SCL/CLC2/C2IN+/AN4/RC0)
- net at U2.11 (RA2/AN2/DACOUT2/C1OUT/T0CKI/~CWG1FLT~/CLC1/PWM3/INT): now also U1.4 (RXD)
- net at J2.5 (Pin_5), U2.12 (RA1/AN1/Vref+/C1IN0-/C2IN0-/ICSPCLK): now also U1.1 (TXD)
- net at U2.2 (RA5/T1CKI/NCO1CLK/CLCIN1/CLKIN): now also U1.6 (~CTS)
- net at U2.3 (RA4/AN3/T1G/NCO1/SDO/CLKOUT): now also U1.2 (~RTS)
- net at U2.6 (CLC2IN1/CWG1B/C2OUT/RC4): now also U3.12 (RCLK); no longer U3.13 (~OE)
- net at U2.7 (~SS~/PWM2/CLCIN0/C2IN3-/C1IN3-/AN7/RC3): now also U3.11 (SRCLK); no longer U3.12 (RCLK)
- net at U2.8 (SDO/C2IN2-/C1IN2-/AN6/RC2): now also U3.14 (SER); no longer U3.11 (SRCLK)
- net at U2.9 (SDI/SDA/PWM4/NCO1/C2IN1-/C1IN1-/AN5/RC1): now also U4.2 (SDA); no longer U3.14 (SER)
- new net: U2.10 (SCK/SCL/CLC2/C2IN+/AN4/RC0), U4.4 (SCL)
- new net: C3.1, D1.2 (A), D2.2 (A), U1.10 (3V3OUT), U1.11 (~RESET), U1.3 (VCCIO)
- new net: R4.1, U1.8 (USBDP)
- new net: R3.1, U1.9 (USBDM)
- new net: J4.1, U4.9 (DSDAM)
- new net: J4.2, U4.8 (DSDAP)
- new net: J4.7, U4.6 (DSCLM)
- new net: J4.8, U4.7 (DSCLP)
- no-connect marks 9 -> 18
Other:
- moved on the sheet: C1, C2, C3, D1, D2, J1, J2, J5, R1, R2, R3, R4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

Commit message: Routed pcb added bom for printer driver
Parts:
- added R10, R13: 120, Resistor_THT:R_Axial_DIN0207_L6.3mm_D2.5mm_P10.16mm_Horizontal, symbol Device:R
- added R11, R12, R14, R9: 600, Resistor_THT:R_Axial_DIN0207_L6.3mm_D2.5mm_P10.16mm_Horizontal, symbol Device:R
- added R7, R8: 2k, Resistor_THT:R_Axial_DIN0207_L6.3mm_D2.5mm_P10.16mm_Horizontal, symbol Device:R
- renumbered J5 to J4, J4 to J5
Connections:
- net +5V: now also R12.1, R7.2, R8.2, R9.1
- net GND: now also R11.2, R14.2
- net at U2.10 (SCK/SCL/CLC2/C2IN+/AN4/RC0), U4.4 (SCL): now also R7.1
- net at U2.9 (SDI/SDA/PWM4/NCO1/C2IN1-/C1IN1-/AN5/RC1), U4.2 (SDA): now also R8.1
- net at J5.1, U4.9 (DSDAM): now also R10.2, R11.1
- net at J5.2, U4.8 (DSDAP): now also R10.1, R9.2
- net at J5.7, U4.6 (DSCLM): now also R13.2, R14.1
- net at J5.8, U4.7 (DSCLP): now also R12.2, R13.1
Other:
- moved on the sheet: J5, U4
