File: Board_Layouts/Front_Panel/Front_Panel.kicad_pcb (KiCad board)
At the start: 2 copper layers, 184 parts, among them J1 Conn_02x18_Odd_Even, SW1 SW_Push_SPDT, SW2 SW_Push, SW3 SW_Push, SW4 SW_SPDT, U1 74LS04, U10 74LS04, U11 74LS154, U12 74LS04, U13 74LS04, U14 HDSP-A401, U2 74LS04, U3 74LS04, U4 7400, U5 74LS121, U6 74LS74, U7 74LS04, U8 74LS04, U9 74LS04

Commit message: Added hex decoders to front panel
Parts:
- added D110: D, Diode_SMD:D_SOD-123, F.Cu at (120.7, -118.1)
- added D111: D, Diode_SMD:D_SOD-123, F.Cu at (100.5, -95.9)
- added D112: D, Diode_SMD:D_SOD-123, F.Cu at (104.3, -124.8)
- added D113: D, Diode_SMD:D_SOD-123, F.Cu at (72.8, -107.4)
- added D114: D, Diode_SMD:D_SOD-123, F.Cu at (66.0, -101.0)
- added D115: D, Diode_SMD:D_SOD-123, F.Cu at (66.0, -97.7)
- added D116: D, Diode_SMD:D_SOD-123, F.Cu at (85.2, -119.4)
- added D117: D, Diode_SMD:D_SOD-123, F.Cu at (98.5, -134.9)
- added D118: D, Diode_SMD:D_SOD-123, F.Cu at (98.5, -131.5)
- added D119: D, Diode_SMD:D_SOD-123, F.Cu at (104.3, -134.9)
- added D120: D, Diode_SMD:D_SOD-123, F.Cu at (91.0, -119.4)
- added D121: D, Diode_SMD:D_SOD-123, F.Cu at (109.2, -111.4)
- added D122: D, Diode_SMD:D_SOD-123, F.Cu at (78.6, -107.4)
- added D123: D, Diode_SMD:D_SOD-123, F.Cu at (91.9, -122.7)
- added D124: D, Diode_SMD:D_SOD-123, F.Cu at (86.2, -116.0)
- added D125: D, Diode_SMD:D_SOD-123, F.Cu at (78.6, -104.0)
- added D126: D, Diode_SMD:D_SOD-123, F.Cu at (86.2, -112.7)
- added D127: D, Diode_SMD:D_SOD-123, F.Cu at (72.8, -104.0)
- added D128: D, Diode_SMD:D_SOD-123, F.Cu at (107.3, -108.1)
- added D129: D, Diode_SMD:D_SOD-123, F.Cu at (101.6, -106.0)
- added D130: D, Diode_SMD:D_SOD-123, F.Cu at (109.2, -114.8)
- added D131: D, Diode_SMD:D_SOD-123, F.Cu at (94.7, -99.3)
- added D132: D, Diode_SMD:D_SOD-123, F.Cu at (121.5, -124.8)
- added D133: D, Diode_SMD:D_SOD-123, F.Cu at (84.3, -102.6)
- added D134: D, Diode_SMD:D_SOD-123, F.Cu at (97.7, -112.7)
- added D135: D, Diode_SMD:D_SOD-123, F.Cu at (71.7, -100.7)
- added D136: D, Diode_SMD:D_SOD-123, F.Cu at (110.0, -134.9)
- added D137: D, Diode_SMD:D_SOD-123, F.Cu at (96.7, -119.4)
- added D138: D, Diode_SMD:D_SOD-123, F.Cu at (77.5, -100.7)
- added D139: D, Diode_SMD:D_SOD-123, F.Cu at (104.3, -128.2)
- added D140: D, Diode_SMD:D_SOD-123, F.Cu at (86.2, -109.3)
- added D141: D, Diode_SMD:D_SOD-123, F.Cu at (91.9, -116.0)
- added D142: D, Diode_SMD:D_SOD-123, F.Cu at (84.3, -106.0)
- added D143: D, Diode_SMD:D_SOD-123, F.Cu at (91.9, -112.7)
- added D144: D, Diode_SMD:D_SOD-123, F.Cu at (71.7, -97.3)
- added D145: D, Diode_SMD:D_SOD-123, F.Cu at (104.3, -131.5)
- added D146: D, Diode_SMD:D_SOD-123, F.Cu at (77.5, -97.3)
- added D147: D, Diode_SMD:D_SOD-123, F.Cu at (110.0, -131.5)
- added D148: D, Diode_SMD:D_SOD-123, F.Cu at (115.8, -134.9)
- added D149: D, Diode_SMD:D_SOD-123, F.Cu at (102.5, -121.5)
- added D150: D, Diode_SMD:D_SOD-123, F.Cu at (110.0, -128.2)
- added D151: D, Diode_SMD:D_SOD-123, F.Cu at (91.9, -109.3)
- added D152: D, Diode_SMD:D_SOD-123, F.Cu at (97.7, -116.0)
- added D153: D, Diode_SMD:D_SOD-123, F.Cu at (90.1, -106.0)
- added D154: D, Diode_SMD:D_SOD-123, F.Cu at (98.5, -128.2)
- added D155: D, Diode_SMD:D_SOD-123, F.Cu at (86.2, -122.7)
- added D156: D, Diode_SMD:D_SOD-123, F.Cu at (113.1, -108.1)
- added D157: D, Diode_SMD:D_SOD-123, F.Cu at (120.7, -114.8)
- added D158: D, Diode_SMD:D_SOD-123, F.Cu at (95.8, -106.0)
- added D159: D, Diode_SMD:D_SOD-123, F.Cu at (110.0, -124.8)
- added D160: D, Diode_SMD:D_SOD-123, F.Cu at (83.2, -99.3)
- added D161: D, Diode_SMD:D_SOD-123, F.Cu at (121.5, -134.9)
- added D162: D, Diode_SMD:D_SOD-123, F.Cu at (108.2, -121.5)
- added D163: D, Diode_SMD:D_SOD-123, F.Cu at (115.8, -128.2)
- added D164: D, Diode_SMD:D_SOD-123, F.Cu at (83.2, -95.9)
- added D165: D, Diode_SMD:D_SOD-123, F.Cu at (90.1, -102.6)
- added D166: D, Diode_SMD:D_SOD-123, F.Cu at (114.9, -118.1)
- added D167: D, Diode_SMD:D_SOD-123, F.Cu at (97.7, -109.3)
- added D168: D, Diode_SMD:D_SOD-123, F.Cu at (115.8, -131.5)
- added D169: D, Diode_SMD:D_SOD-123, F.Cu at (103.4, -114.8)
- added D170: D, Diode_SMD:D_SOD-123, F.Cu at (89.0, -99.3)
- added D171: D, Diode_SMD:D_SOD-123, F.Cu at (121.5, -131.5)
- added D172: D, Diode_SMD:D_SOD-123, F.Cu at (115.8, -124.8)
- added D173: D, Diode_SMD:D_SOD-123, F.Cu at (103.4, -111.4)
- added D174: D, Diode_SMD:D_SOD-123, F.Cu at (109.2, -118.1)
- added D175: D, Diode_SMD:D_SOD-123, F.Cu at (114.0, -121.5)
- added D176: D, Diode_SMD:D_SOD-123, F.Cu at (121.5, -128.2)
- added D177: D, Diode_SMD:D_SOD-123, F.Cu at (89.0, -95.9)
- added D178: D, Diode_SMD:D_SOD-123, F.Cu at (103.4, -118.1)
- added D179: D, Diode_SMD:D_SOD-123, F.Cu at (98.5, -124.8)
- added D180: D, Diode_SMD:D_SOD-123, F.Cu at (119.7, -121.5)
- added D181: D, Diode_SMD:D_SOD-123, F.Cu at (94.7, -95.9)
- added D182: D, Diode_SMD:D_SOD-123, F.Cu at (101.6, -102.6)
- added D183: D, Diode_SMD:D_SOD-123, F.Cu at (95.8, -102.6)
- added D184: D, Diode_SMD:D_SOD-123, F.Cu at (114.9, -114.8)
- added D185: D, Diode_SMD:D_SOD-123, F.Cu at (100.5, -99.3)
- added D186: D, Diode_SMD:D_SOD-123, F.Cu at (114.9, -111.4)
- added D187: D, Diode_SMD:D_SOD-123, F.Cu at (107.3, -104.7)
- added D188: D, Diode_SMD:D_SOD-123, F.Cu at (107.3, -61.5)
- added D189: D, Diode_SMD:D_SOD-123, F.Cu at (85.2, -72.8)
- added D190: D, Diode_SMD:D_SOD-123, F.Cu at (98.5, -88.3)
- added D191: D, Diode_SMD:D_SOD-123, F.Cu at (98.5, -85.0)
- added D192: D, Diode_SMD:D_SOD-123, F.Cu at (104.3, -88.3)
- added D193: D, Diode_SMD:D_SOD-123, F.Cu at (91.0, -72.8)
- added D194: D, Diode_SMD:D_SOD-123, F.Cu at (98.5, -81.6)
- added D195: D, Diode_SMD:D_SOD-123, F.Cu at (78.6, -60.8)
- added D196: D, Diode_SMD:D_SOD-123, F.Cu at (91.9, -76.2)
- added D197: D, Diode_SMD:D_SOD-123, F.Cu at (86.2, -69.5)
- added D198: D, Diode_SMD:D_SOD-123, F.Cu at (78.6, -57.5)
- added D199: D, Diode_SMD:D_SOD-123, F.Cu at (86.2, -66.1)
- added D200: D, Diode_SMD:D_SOD-123, F.Cu at (98.5, -78.3)
- added D201: D, Diode_SMD:D_SOD-123, F.Cu at (114.9, -68.2)
- added D202: D, Diode_SMD:D_SOD-123, F.Cu at (66.0, -51.2)
- added D203: D, Diode_SMD:D_SOD-123, F.Cu at (101.6, -59.4)
- added D204: D, Diode_SMD:D_SOD-123, F.Cu at (109.2, -68.2)
- added D205: D, Diode_SMD:D_SOD-123, F.Cu at (94.7, -52.7)
- added D206: D, Diode_SMD:D_SOD-123, F.Cu at (121.5, -78.3)
- added D207: D, Diode_SMD:D_SOD-123, F.Cu at (109.2, -64.9)
- added D208: D, Diode_SMD:D_SOD-123, F.Cu at (71.7, -54.1)
- added D209: D, Diode_SMD:D_SOD-123, F.Cu at (119.7, -74.9)
- added D210: D, Diode_SMD:D_SOD-123, F.Cu at (94.7, -49.4)
- added D211: D, Diode_SMD:D_SOD-123, F.Cu at (101.6, -56.1)
- added D212: D, Diode_SMD:D_SOD-123, F.Cu at (95.8, -56.1)
- added D213: D, Diode_SMD:D_SOD-123, F.Cu at (110.0, -88.3)
- added D214: D, Diode_SMD:D_SOD-123, F.Cu at (86.2, -76.2)
- added D215: D, Diode_SMD:D_SOD-123, F.Cu at (110.0, -78.3)
- added D216: D, Diode_SMD:D_SOD-123, F.Cu at (77.5, -54.1)
- added D217: D, Diode_SMD:D_SOD-123, F.Cu at (104.3, -81.6)
- added D218: D, Diode_SMD:D_SOD-123, F.Cu at (86.2, -62.8)
- added D219: D, Diode_SMD:D_SOD-123, F.Cu at (91.9, -69.5)
- added D220: D, Diode_SMD:D_SOD-123, F.Cu at (84.3, -59.4)
- added D221: D, Diode_SMD:D_SOD-123, F.Cu at (91.9, -66.1)
- added D222: D, Diode_SMD:D_SOD-123, F.Cu at (104.3, -78.3)
- added D223: D, Diode_SMD:D_SOD-123, F.Cu at (102.5, -74.9)
- added D224: D, Diode_SMD:D_SOD-123, F.Cu at (91.9, -62.8)
- added D225: D, Diode_SMD:D_SOD-123, F.Cu at (84.3, -56.1)
- added D226: D, Diode_SMD:D_SOD-123, F.Cu at (97.7, -69.5)
- added D227: D, Diode_SMD:D_SOD-123, F.Cu at (90.1, -59.4)
- added D228: D, Diode_SMD:D_SOD-123, F.Cu at (97.7, -66.1)
- added D229: D, Diode_SMD:D_SOD-123, F.Cu at (77.5, -50.8)
- added D230: D, Diode_SMD:D_SOD-123, F.Cu at (72.8, -60.8)
- added D231: D, Diode_SMD:D_SOD-123, F.Cu at (66.0, -54.5)
- added D232: D, Diode_SMD:D_SOD-123, F.Cu at (72.8, -57.5)
- added D233: D, Diode_SMD:D_SOD-123, F.Cu at (110.0, -81.6)
- added D234: D, Diode_SMD:D_SOD-123, F.Cu at (115.8, -88.3)
- added D235: D, Diode_SMD:D_SOD-123, F.Cu at (110.0, -85.0)
- added D236: D, Diode_SMD:D_SOD-123, F.Cu at (71.7, -50.8)
- added D237: D, Diode_SMD:D_SOD-123, F.Cu at (104.3, -85.0)
- added D238: D, Diode_SMD:D_SOD-123, F.Cu at (96.7, -72.8)
- added D239: D, Diode_SMD:D_SOD-123, F.Cu at (103.4, -71.6)
- added D240: D, Diode_SMD:D_SOD-123, F.Cu at (83.2, -52.7)
- added D241: D, Diode_SMD:D_SOD-123, F.Cu at (121.5, -88.3)
- added D242: D, Diode_SMD:D_SOD-123, F.Cu at (108.2, -74.9)
- added D243: D, Diode_SMD:D_SOD-123, F.Cu at (115.8, -81.6)
- added D244: D, Diode_SMD:D_SOD-123, F.Cu at (83.2, -49.4)
- added D245: D, Diode_SMD:D_SOD-123, F.Cu at (90.1, -56.1)
- added D246: D, Diode_SMD:D_SOD-123, F.Cu at (97.7, -62.8)
- added D247: D, Diode_SMD:D_SOD-123, F.Cu at (115.8, -85.0)
- added D248: D, Diode_SMD:D_SOD-123, F.Cu at (103.4, -68.2)
- added D249: D, Diode_SMD:D_SOD-123, F.Cu at (114.9, -71.6)
- added D250: D, Diode_SMD:D_SOD-123, F.Cu at (89.0, -49.4)
- added D251: D, Diode_SMD:D_SOD-123, F.Cu at (121.5, -81.6)
- added D252: D, Diode_SMD:D_SOD-123, F.Cu at (109.2, -71.6)
- added D253: D, Diode_SMD:D_SOD-123, F.Cu at (103.4, -64.9)
- added D254: D, Diode_SMD:D_SOD-123, F.Cu at (115.8, -78.3)
- added D255: D, Diode_SMD:D_SOD-123, F.Cu at (121.5, -85.0)
- added D256: D, Diode_SMD:D_SOD-123, F.Cu at (89.0, -52.7)
- added D257: D, Diode_SMD:D_SOD-123, F.Cu at (114.0, -74.9)
- added D258: D, Diode_SMD:D_SOD-123, F.Cu at (95.8, -59.4)
- added D259: D, Diode_SMD:D_SOD-123, F.Cu at (100.5, -52.7)
- added D260: D, Diode_SMD:D_SOD-123, F.Cu at (114.9, -64.9)
- added D261: D, Diode_SMD:D_SOD-123, F.Cu at (107.3, -58.2)
- added D262: D, Diode_SMD:D_SOD-123, F.Cu at (120.7, -71.6)
- added D263: D, Diode_SMD:D_SOD-123, F.Cu at (100.5, -49.4)
- added D264: D, Diode_SMD:D_SOD-123, F.Cu at (113.1, -61.5)
- added D265: D, Diode_SMD:D_SOD-123, F.Cu at (120.7, -68.2)
- added D266: D, Diode_SMD:D_SOD-123, F.Cu at (178.9, -128.2)
- added D267: D, Diode_SMD:D_SOD-123, F.Cu at (159.0, -107.4)
- added D268: D, Diode_SMD:D_SOD-123, F.Cu at (172.3, -122.7)
- added D269: D, Diode_SMD:D_SOD-123, F.Cu at (166.5, -116.0)
- added D270: D, Diode_SMD:D_SOD-123, F.Cu at (159.0, -104.0)
- added D271: D, Diode_SMD:D_SOD-123, F.Cu at (166.5, -112.7)
- added D272: D, Diode_SMD:D_SOD-123, F.Cu at (178.9, -124.8)
- added D273: D, Diode_SMD:D_SOD-123, F.Cu at (184.7, -131.5)
- added D274: D, Diode_SMD:D_SOD-123, F.Cu at (152.1, -100.7)
- added D275: D, Diode_SMD:D_SOD-123, F.Cu at (152.1, -97.3)
- added D276: D, Diode_SMD:D_SOD-123, F.Cu at (187.7, -108.1)
- added D277: D, Diode_SMD:D_SOD-123, F.Cu at (182.0, -106.0)
- added D278: D, Diode_SMD:D_SOD-123, F.Cu at (193.5, -108.1)
- added D279: D, Diode_SMD:D_SOD-123, F.Cu at (175.1, -99.3)
- added D280: D, Diode_SMD:D_SOD-123, F.Cu at (201.9, -124.8)
- added D281: D, Diode_SMD:D_SOD-123, F.Cu at (189.5, -111.4)
- added D282: D, Diode_SMD:D_SOD-123, F.Cu at (170.5, -106.0)
- added D283: D, Diode_SMD:D_SOD-123, F.Cu at (200.1, -121.5)
- added D284: D, Diode_SMD:D_SOD-123, F.Cu at (175.1, -95.9)
- added D285: D, Diode_SMD:D_SOD-123, F.Cu at (182.0, -102.6)
- added D286: D, Diode_SMD:D_SOD-123, F.Cu at (176.2, -102.6)
- added D287: D, Diode_SMD:D_SOD-123, F.Cu at (195.3, -114.8)
- added D288: D, Diode_SMD:D_SOD-123, F.Cu at (180.9, -99.3)
- added D289: D, Diode_SMD:D_SOD-123, F.Cu at (195.3, -111.4)
- added D290: D, Diode_SMD:D_SOD-123, F.Cu at (187.7, -104.7)
- added D291: D, Diode_SMD:D_SOD-123, F.Cu at (201.0, -118.1)
- added D292: D, Diode_SMD:D_SOD-123, F.Cu at (180.9, -95.9)
- added D293: D, Diode_SMD:D_SOD-123, F.Cu at (182.9, -121.5)
- added D294: D, Diode_SMD:D_SOD-123, F.Cu at (184.7, -134.9)
- added D295: D, Diode_SMD:D_SOD-123, F.Cu at (196.2, -134.9)
- added D296: D, Diode_SMD:D_SOD-123, F.Cu at (190.4, -134.9)
- added D297: D, Diode_SMD:D_SOD-123, F.Cu at (157.9, -97.3)
- added D298: D, Diode_SMD:D_SOD-123, F.Cu at (184.7, -124.8)
- added D299: D, Diode_SMD:D_SOD-123, F.Cu at (172.3, -112.7)
- added D300: D, Diode_SMD:D_SOD-123, F.Cu at (164.7, -106.0)
- added D301: D, Diode_SMD:D_SOD-123, F.Cu at (172.3, -116.0)
- added D302: D, Diode_SMD:D_SOD-123, F.Cu at (166.5, -109.3)
- added D303: D, Diode_SMD:D_SOD-123, F.Cu at (190.4, -128.2)
- added D304: D, Diode_SMD:D_SOD-123, F.Cu at (184.7, -128.2)
- added D305: D, Diode_SMD:D_SOD-123, F.Cu at (157.9, -100.7)
- added D306: D, Diode_SMD:D_SOD-123, F.Cu at (177.1, -119.4)
- added D307: D, Diode_SMD:D_SOD-123, F.Cu at (172.3, -109.3)
- added D308: D, Diode_SMD:D_SOD-123, F.Cu at (164.7, -102.6)
- added D309: D, Diode_SMD:D_SOD-123, F.Cu at (178.0, -116.0)
- added D310: D, Diode_SMD:D_SOD-123, F.Cu at (165.6, -119.4)
- added D311: D, Diode_SMD:D_SOD-123, F.Cu at (178.0, -112.7)
- added D312: D, Diode_SMD:D_SOD-123, F.Cu at (190.4, -131.5)
- added D313: D, Diode_SMD:D_SOD-123, F.Cu at (153.2, -107.4)
- added D314: D, Diode_SMD:D_SOD-123, F.Cu at (146.4, -101.0)
- added D315: D, Diode_SMD:D_SOD-123, F.Cu at (153.2, -104.0)
- added D316: D, Diode_SMD:D_SOD-123, F.Cu at (146.4, -97.7)
- added D317: D, Diode_SMD:D_SOD-123, F.Cu at (166.5, -122.7)
- added D318: D, Diode_SMD:D_SOD-123, F.Cu at (178.9, -134.9)
- added D319: D, Diode_SMD:D_SOD-123, F.Cu at (178.9, -131.5)
- added D320: D, Diode_SMD:D_SOD-123, F.Cu at (189.5, -114.8)
- added D321: D, Diode_SMD:D_SOD-123, F.Cu at (171.4, -119.4)
- added D322: D, Diode_SMD:D_SOD-123, F.Cu at (195.3, -118.1)
- added D323: D, Diode_SMD:D_SOD-123, F.Cu at (196.2, -128.2)
- added D324: D, Diode_SMD:D_SOD-123, F.Cu at (163.6, -95.9)
- added D325: D, Diode_SMD:D_SOD-123, F.Cu at (170.5, -102.6)
- added D326: D, Diode_SMD:D_SOD-123, F.Cu at (183.8, -118.1)
- added D327: D, Diode_SMD:D_SOD-123, F.Cu at (178.0, -109.3)
- added D328: D, Diode_SMD:D_SOD-123, F.Cu at (196.2, -131.5)
- added D329: D, Diode_SMD:D_SOD-123, F.Cu at (183.8, -114.8)
- added D330: D, Diode_SMD:D_SOD-123, F.Cu at (169.4, -99.3)
- added D331: D, Diode_SMD:D_SOD-123, F.Cu at (201.9, -131.5)
- added D332: D, Diode_SMD:D_SOD-123, F.Cu at (188.6, -121.5)
- added D333: D, Diode_SMD:D_SOD-123, F.Cu at (196.2, -124.8)
- added D334: D, Diode_SMD:D_SOD-123, F.Cu at (169.4, -95.9)
- added D335: D, Diode_SMD:D_SOD-123, F.Cu at (201.9, -128.2)
- added D336: D, Diode_SMD:D_SOD-123, F.Cu at (194.4, -121.5)
- added D337: D, Diode_SMD:D_SOD-123, F.Cu at (189.5, -118.1)
- added D338: D, Diode_SMD:D_SOD-123, F.Cu at (183.8, -111.4)
- added D339: D, Diode_SMD:D_SOD-123, F.Cu at (201.9, -134.9)
- added D340: D, Diode_SMD:D_SOD-123, F.Cu at (201.0, -114.8)
- added D341: D, Diode_SMD:D_SOD-123, F.Cu at (176.2, -106.0)
- added D342: D, Diode_SMD:D_SOD-123, F.Cu at (190.4, -124.8)
- added D343: D, Diode_SMD:D_SOD-123, F.Cu at (163.6, -99.3)
- added D344: D, Diode_SMD:D_SOD-123, F.Cu at (178.9, -81.6)
- added D345: D, Diode_SMD:D_SOD-123, F.Cu at (159.0, -60.8)
- added D346: D, Diode_SMD:D_SOD-123, F.Cu at (172.3, -76.2)
- added D347: D, Diode_SMD:D_SOD-123, F.Cu at (166.5, -69.5)
- added D348: D, Diode_SMD:D_SOD-123, F.Cu at (159.0, -57.5)
- added D349: D, Diode_SMD:D_SOD-123, F.Cu at (166.5, -66.1)
- added D350: D, Diode_SMD:D_SOD-123, F.Cu at (178.9, -78.3)
- added D351: D, Diode_SMD:D_SOD-123, F.Cu at (184.7, -85.0)
- added D352: D, Diode_SMD:D_SOD-123, F.Cu at (152.1, -54.1)
- added D353: D, Diode_SMD:D_SOD-123, F.Cu at (178.9, -88.3)
- added D354: D, Diode_SMD:D_SOD-123, F.Cu at (187.7, -61.5)
- added D355: D, Diode_SMD:D_SOD-123, F.Cu at (182.0, -59.4)
- added D356: D, Diode_SMD:D_SOD-123, F.Cu at (189.5, -68.2)
- added D357: D, Diode_SMD:D_SOD-123, F.Cu at (175.1, -52.7)
- added D358: D, Diode_SMD:D_SOD-123, F.Cu at (201.9, -78.3)
- added D359: D, Diode_SMD:D_SOD-123, F.Cu at (195.3, -64.9)
- added D360: D, Diode_SMD:D_SOD-123, F.Cu at (163.6, -52.7)
- added D361: D, Diode_SMD:D_SOD-123, F.Cu at (190.4, -78.3)
- added D362: D, Diode_SMD:D_SOD-123, F.Cu at (176.2, -59.4)
- added D363: D, Diode_SMD:D_SOD-123, F.Cu at (201.0, -68.2)
- added D364: D, Diode_SMD:D_SOD-123, F.Cu at (193.5, -61.5)
- added D365: D, Diode_SMD:D_SOD-123, F.Cu at (180.9, -49.4)
- added D366: D, Diode_SMD:D_SOD-123, F.Cu at (201.0, -71.6)
- added D367: D, Diode_SMD:D_SOD-123, F.Cu at (187.7, -58.2)
- added D368: D, Diode_SMD:D_SOD-123, F.Cu at (201.9, -88.3)
- added D369: D, Diode_SMD:D_SOD-123, F.Cu at (180.9, -52.7)
- added D370: D, Diode_SMD:D_SOD-123, F.Cu at (195.3, -68.2)
- added D371: D, Diode_SMD:D_SOD-123, F.Cu at (176.2, -56.1)
- added D372: D, Diode_SMD:D_SOD-123, F.Cu at (189.5, -64.9)
- added D373: D, Diode_SMD:D_SOD-123, F.Cu at (175.1, -49.4)
- added D374: D, Diode_SMD:D_SOD-123, F.Cu at (200.1, -74.9)
- added D375: D, Diode_SMD:D_SOD-123, F.Cu at (152.1, -50.8)
- added D376: D, Diode_SMD:D_SOD-123, F.Cu at (184.7, -81.6)
- added D377: D, Diode_SMD:D_SOD-123, F.Cu at (177.1, -72.8)
- added D378: D, Diode_SMD:D_SOD-123, F.Cu at (157.9, -54.1)
- added D379: D, Diode_SMD:D_SOD-123, F.Cu at (184.7, -78.3)
- added D380: D, Diode_SMD:D_SOD-123, F.Cu at (196.2, -88.3)
- added D381: D, Diode_SMD:D_SOD-123, F.Cu at (182.9, -74.9)
- added D382: D, Diode_SMD:D_SOD-123, F.Cu at (190.4, -81.6)
- added D383: D, Diode_SMD:D_SOD-123, F.Cu at (171.4, -72.8)
- added D384: D, Diode_SMD:D_SOD-123, F.Cu at (172.3, -62.8)
- added D385: D, Diode_SMD:D_SOD-123, F.Cu at (164.7, -56.1)
- added D386: D, Diode_SMD:D_SOD-123, F.Cu at (178.0, -69.5)
- added D387: D, Diode_SMD:D_SOD-123, F.Cu at (170.5, -59.4)
- added D388: D, Diode_SMD:D_SOD-123, F.Cu at (146.4, -54.5)
- added D389: D, Diode_SMD:D_SOD-123, F.Cu at (153.2, -57.5)
- added D390: D, Diode_SMD:D_SOD-123, F.Cu at (146.4, -51.2)
- added D391: D, Diode_SMD:D_SOD-123, F.Cu at (165.6, -72.8)
- added D392: D, Diode_SMD:D_SOD-123, F.Cu at (166.5, -76.2)
- added D393: D, Diode_SMD:D_SOD-123, F.Cu at (178.9, -85.0)
- added D394: D, Diode_SMD:D_SOD-123, F.Cu at (184.7, -88.3)
- added D395: D, Diode_SMD:D_SOD-123, F.Cu at (153.2, -60.8)
- added D396: D, Diode_SMD:D_SOD-123, F.Cu at (190.4, -85.0)
- added D397: D, Diode_SMD:D_SOD-123, F.Cu at (178.0, -66.1)
- added D398: D, Diode_SMD:D_SOD-123, F.Cu at (190.4, -88.3)
- added D399: D, Diode_SMD:D_SOD-123, F.Cu at (157.9, -50.8)
- added D400: D, Diode_SMD:D_SOD-123, F.Cu at (172.3, -66.1)
- added D401: D, Diode_SMD:D_SOD-123, F.Cu at (164.7, -59.4)
- added D402: D, Diode_SMD:D_SOD-123, F.Cu at (172.3, -69.5)
- added D403: D, Diode_SMD:D_SOD-123, F.Cu at (166.5, -62.8)
- added D404: D, Diode_SMD:D_SOD-123, F.Cu at (188.6, -74.9)
- added D405: D, Diode_SMD:D_SOD-123, F.Cu at (182.0, -56.1)
- added D406: D, Diode_SMD:D_SOD-123, F.Cu at (183.8, -71.6)
- added D407: D, Diode_SMD:D_SOD-123, F.Cu at (178.0, -62.8)
- added D408: D, Diode_SMD:D_SOD-123, F.Cu at (196.2, -85.0)
- added D409: D, Diode_SMD:D_SOD-123, F.Cu at (183.8, -68.2)
- added D410: D, Diode_SMD:D_SOD-123, F.Cu at (169.4, -52.7)
- added D411: D, Diode_SMD:D_SOD-123, F.Cu at (201.9, -85.0)
- added D412: D, Diode_SMD:D_SOD-123, F.Cu at (196.2, -78.3)
- added D413: D, Diode_SMD:D_SOD-123, F.Cu at (169.4, -49.4)
- added D414: D, Diode_SMD:D_SOD-123, F.Cu at (201.9, -81.6)
- added D415: D, Diode_SMD:D_SOD-123, F.Cu at (194.4, -74.9)
- added D416: D, Diode_SMD:D_SOD-123, F.Cu at (189.5, -71.6)
- added D417: D, Diode_SMD:D_SOD-123, F.Cu at (183.8, -64.9)
- added D418: D, Diode_SMD:D_SOD-123, F.Cu at (195.3, -71.6)
- added D419: D, Diode_SMD:D_SOD-123, F.Cu at (170.5, -56.1)
- added D420: D, Diode_SMD:D_SOD-123, F.Cu at (163.6, -49.4)
- added D421: D, Diode_SMD:D_SOD-123, F.Cu at (196.2, -81.6)
- added D422: D, Diode_SMD:D_SOD-123, F.Cu at (256.6, -102.6)
- added D423: D, Diode_SMD:D_SOD-123, F.Cu at (262.4, -102.6)
- added D424: D, Diode_SMD:D_SOD-123, F.Cu at (255.5, -95.9)
- added D425: D, Diode_SMD:D_SOD-123, F.Cu at (280.5, -121.5)
- added D426: D, Diode_SMD:D_SOD-123, F.Cu at (252.7, -109.3)
- added D427: D, Diode_SMD:D_SOD-123, F.Cu at (269.9, -111.4)
- added D428: D, Diode_SMD:D_SOD-123, F.Cu at (282.3, -124.8)
- added D429: D, Diode_SMD:D_SOD-123, F.Cu at (255.5, -99.3)
- added D430: D, Diode_SMD:D_SOD-123, F.Cu at (275.7, -114.8)
- added D431: D, Diode_SMD:D_SOD-123, F.Cu at (262.4, -106.0)
- added D432: D, Diode_SMD:D_SOD-123, F.Cu at (268.1, -108.1)
- added D433: D, Diode_SMD:D_SOD-123, F.Cu at (232.5, -97.3)
- added D434: D, Diode_SMD:D_SOD-123, F.Cu at (232.5, -100.7)
- added D435: D, Diode_SMD:D_SOD-123, F.Cu at (265.1, -131.5)
- added D436: D, Diode_SMD:D_SOD-123, F.Cu at (259.3, -124.8)
- added D437: D, Diode_SMD:D_SOD-123, F.Cu at (246.9, -112.7)
- added D438: D, Diode_SMD:D_SOD-123, F.Cu at (256.6, -106.0)
- added D439: D, Diode_SMD:D_SOD-123, F.Cu at (264.2, -118.1)
- added D440: D, Diode_SMD:D_SOD-123, F.Cu at (250.8, -102.6)
- added D441: D, Diode_SMD:D_SOD-123, F.Cu at (244.0, -95.9)
- added D442: D, Diode_SMD:D_SOD-123, F.Cu at (276.6, -128.2)
- added D443: D, Diode_SMD:D_SOD-123, F.Cu at (269.0, -121.5)
- added D444: D, Diode_SMD:D_SOD-123, F.Cu at (282.3, -134.9)
- added D445: D, Diode_SMD:D_SOD-123, F.Cu at (244.0, -99.3)
- added D446: D, Diode_SMD:D_SOD-123, F.Cu at (270.8, -124.8)
- added D447: D, Diode_SMD:D_SOD-123, F.Cu at (258.4, -109.3)
- added D448: D, Diode_SMD:D_SOD-123, F.Cu at (281.4, -114.8)
- added D449: D, Diode_SMD:D_SOD-123, F.Cu at (273.9, -108.1)
- added D450: D, Diode_SMD:D_SOD-123, F.Cu at (261.2, -95.9)
- added D451: D, Diode_SMD:D_SOD-123, F.Cu at (281.4, -118.1)
- added D452: D, Diode_SMD:D_SOD-123, F.Cu at (268.1, -104.7)
- added D453: D, Diode_SMD:D_SOD-123, F.Cu at (275.7, -111.4)
- added D454: D, Diode_SMD:D_SOD-123, F.Cu at (261.2, -99.3)
- added D455: D, Diode_SMD:D_SOD-123, F.Cu at (269.9, -114.8)
- added D456: D, Diode_SMD:D_SOD-123, F.Cu at (257.5, -119.4)
- added D457: D, Diode_SMD:D_SOD-123, F.Cu at (238.2, -100.7)
- added D458: D, Diode_SMD:D_SOD-123, F.Cu at (265.1, -128.2)
- added D459: D, Diode_SMD:D_SOD-123, F.Cu at (246.9, -109.3)
- added D460: D, Diode_SMD:D_SOD-123, F.Cu at (252.7, -116.0)
- added D461: D, Diode_SMD:D_SOD-123, F.Cu at (245.1, -106.0)
- added D462: D, Diode_SMD:D_SOD-123, F.Cu at (252.7, -112.7)
- added D463: D, Diode_SMD:D_SOD-123, F.Cu at (265.1, -124.8)
- added D464: D, Diode_SMD:D_SOD-123, F.Cu at (238.2, -97.3)
- added D465: D, Diode_SMD:D_SOD-123, F.Cu at (270.8, -134.9)
- added D466: D, Diode_SMD:D_SOD-123, F.Cu at (276.6, -134.9)
- added D467: D, Diode_SMD:D_SOD-123, F.Cu at (263.2, -121.5)
- added D468: D, Diode_SMD:D_SOD-123, F.Cu at (270.8, -128.2)
- added D469: D, Diode_SMD:D_SOD-123, F.Cu at (251.7, -119.4)
- added D470: D, Diode_SMD:D_SOD-123, F.Cu at (245.1, -102.6)
- added D471: D, Diode_SMD:D_SOD-123, F.Cu at (246.0, -119.4)
- added D472: D, Diode_SMD:D_SOD-123, F.Cu at (246.9, -116.0)
- added D473: D, Diode_SMD:D_SOD-123, F.Cu at (252.7, -122.7)
- added D474: D, Diode_SMD:D_SOD-123, F.Cu at (239.3, -107.4)
- added D475: D, Diode_SMD:D_SOD-123, F.Cu at (259.3, -128.2)
- added D476: D, Diode_SMD:D_SOD-123, F.Cu at (233.6, -107.4)
- added D477: D, Diode_SMD:D_SOD-123, F.Cu at (226.8, -101.0)
- added D478: D, Diode_SMD:D_SOD-123, F.Cu at (233.6, -104.0)
- added D479: D, Diode_SMD:D_SOD-123, F.Cu at (226.8, -97.7)
- added D480: D, Diode_SMD:D_SOD-123, F.Cu at (239.3, -104.0)
- added D481: D, Diode_SMD:D_SOD-123, F.Cu at (259.3, -134.9)
- added D482: D, Diode_SMD:D_SOD-123, F.Cu at (259.3, -131.5)
- added D483: D, Diode_SMD:D_SOD-123, F.Cu at (265.1, -134.9)
- added D484: D, Diode_SMD:D_SOD-123, F.Cu at (246.9, -122.7)
- added D485: D, Diode_SMD:D_SOD-123, F.Cu at (270.8, -131.5)
- added D486: D, Diode_SMD:D_SOD-123, F.Cu at (258.4, -112.7)
- added D487: D, Diode_SMD:D_SOD-123, F.Cu at (250.8, -106.0)
- added D488: D, Diode_SMD:D_SOD-123, F.Cu at (258.4, -116.0)
- added D489: D, Diode_SMD:D_SOD-123, F.Cu at (275.7, -118.1)
- added D490: D, Diode_SMD:D_SOD-123, F.Cu at (249.8, -95.9)
- added D491: D, Diode_SMD:D_SOD-123, F.Cu at (282.3, -128.2)
- added D492: D, Diode_SMD:D_SOD-123, F.Cu at (274.7, -121.5)
- added D493: D, Diode_SMD:D_SOD-123, F.Cu at (264.2, -114.8)
- added D494: D, Diode_SMD:D_SOD-123, F.Cu at (249.8, -99.3)
- added D495: D, Diode_SMD:D_SOD-123, F.Cu at (282.3, -131.5)
- added D496: D, Diode_SMD:D_SOD-123, F.Cu at (276.6, -124.8)
- added D497: D, Diode_SMD:D_SOD-123, F.Cu at (264.2, -111.4)
- added D498: D, Diode_SMD:D_SOD-123, F.Cu at (269.9, -118.1)
- added D499: D, Diode_SMD:D_SOD-123, F.Cu at (276.6, -131.5)
- added R46: 330, Resistor_THT:R_Axial_DIN0207_L6.3mm_D2.5mm_P10.16mm_Horizontal, F.Cu at (71.5, -115.1)
- added R47: 330, Resistor_THT:R_Axial_DIN0207_L6.3mm_D2.5mm_P10.16mm_Horizontal, F.Cu at (71.5, -111.1)
- added R48: 330, Resistor_THT:R_Axial_DIN0207_L6.3mm_D2.5mm_P10.16mm_Horizontal, F.Cu at (83.9, -126.4)
- added R49: 330, Resistor_THT:R_Axial_DIN0207_L6.3mm_D2.5mm_P10.16mm_Horizontal, F.Cu at (51.4, -96.7)
- added R50: 330, Resistor_THT:R_Axial_DIN0207_L6.3mm_D2.5mm_P10.16mm_Horizontal, F.Cu at (51.4, -100.7)
- added R51: 330, Resistor_THT:R_Axial_DIN0207_L6.3mm_D2.5mm_P10.16mm_Horizontal, F.Cu at (83.9, -130.5)
- added R52: 330, Resistor_THT:R_Axial_DIN0207_L6.3mm_D2.5mm_P10.16mm_Horizontal, F.Cu at (83.9, -134.5)
- added R53: 330, Resistor_THT:R_Axial_DIN0207_L6.3mm_D2.5mm_P10.16mm_Horizontal, F.Cu at (71.5, -64.5)
- added R54: 330, Resistor_THT:R_Axial_DIN0207_L6.3mm_D2.5mm_P10.16mm_Horizontal, F.Cu at (83.9, -79.9)
- added R55: 330, Resistor_THT:R_Axial_DIN0207_L6.3mm_D2.5mm_P10.16mm_Horizontal, F.Cu at (51.4, -50.1)
- added R56: 330, Resistor_THT:R_Axial_DIN0207_L6.3mm_D2.5mm_P10.16mm_Horizontal, F.Cu at (51.4, -54.2)
- added R57: 330, Resistor_THT:R_Axial_DIN0207_L6.3mm_D2.5mm_P10.16mm_Horizontal, F.Cu at (83.9, -83.9)
- added R58: 330, Resistor_THT:R_Axial_DIN0207_L6.3mm_D2.5mm_P10.16mm_Horizontal, F.Cu at (83.9, -88.0)
- added R59: 330, Resistor_THT:R_Axial_DIN0207_L6.3mm_D2.5mm_P10.16mm_Horizontal, F.Cu at (71.5, -68.6)
- added R60: 330, Resistor_THT:R_Axial_DIN0207_L6.3mm_D2.5mm_P10.16mm_Horizontal, F.Cu at (151.9, -115.1)
- added R61: 330, Resistor_THT:R_Axial_DIN0207_L6.3mm_D2.5mm_P10.16mm_Horizontal, F.Cu at (164.3, -134.5)
- added R62: 330, Resistor_THT:R_Axial_DIN0207_L6.3mm_D2.5mm_P10.16mm_Horizontal, F.Cu at (164.3, -130.5)
- added R63: 330, Resistor_THT:R_Axial_DIN0207_L6.3mm_D2.5mm_P10.16mm_Horizontal, F.Cu at (151.9, -111.1)
- added R64: 330, Resistor_THT:R_Axial_DIN0207_L6.3mm_D2.5mm_P10.16mm_Horizontal, F.Cu at (131.8, -100.7)
- added R65: 330, Resistor_THT:R_Axial_DIN0207_L6.3mm_D2.5mm_P10.16mm_Horizontal, F.Cu at (131.8, -96.7)
- added R66: 330, Resistor_THT:R_Axial_DIN0207_L6.3mm_D2.5mm_P10.16mm_Horizontal, F.Cu at (164.3, -126.4)
- added R67: 330, Resistor_THT:R_Axial_DIN0207_L6.3mm_D2.5mm_P10.16mm_Horizontal, F.Cu at (151.9, -68.6)
- added R68: 330, Resistor_THT:R_Axial_DIN0207_L6.3mm_D2.5mm_P10.16mm_Horizontal, F.Cu at (164.3, -88.0)
- added R69: 330, Resistor_THT:R_Axial_DIN0207_L6.3mm_D2.5mm_P10.16mm_Horizontal, F.Cu at (164.3, -83.9)
- added R70: 330, Resistor_THT:R_Axial_DIN0207_L6.3mm_D2.5mm_P10.16mm_Horizontal, F.Cu at (131.8, -54.2)
- added R71: 330, Resistor_THT:R_Axial_DIN0207_L6.3mm_D2.5mm_P10.16mm_Horizontal, F.Cu at (131.8, -50.1)
- added R72: 330, Resistor_THT:R_Axial_DIN0207_L6.3mm_D2.5mm_P10.16mm_Horizontal, F.Cu at (164.3, -79.9)
- added R73: 330, Resistor_THT:R_Axial_DIN0207_L6.3mm_D2.5mm_P10.16mm_Horizontal, F.Cu at (151.9, -64.5)
- added R74: 330, Resistor_THT:R_Axial_DIN0207_L6.3mm_D2.5mm_P10.16mm_Horizontal, F.Cu at (232.3, -111.1)
- added R75: 330, Resistor_THT:R_Axial_DIN0207_L6.3mm_D2.5mm_P10.16mm_Horizontal, F.Cu at (244.7, -126.4)
- added R76: 330, Resistor_THT:R_Axial_DIN0207_L6.3mm_D2.5mm_P10.16mm_Horizontal, F.Cu at (232.3, -115.1)
- added R77: 330, Resistor_THT:R_Axial_DIN0207_L6.3mm_D2.5mm_P10.16mm_Horizontal, F.Cu at (212.1, -96.7)
- added R78: 330, Resistor_THT:R_Axial_DIN0207_L6.3mm_D2.5mm_P10.16mm_Horizontal, F.Cu at (212.1, -100.7)
- added R79: 330, Resistor_THT:R_Axial_DIN0207_L6.3mm_D2.5mm_P10.16mm_Horizontal, F.Cu at (244.7, -130.5)
- added R80: 330, Resistor_THT:R_Axial_DIN0207_L6.3mm_D2.5mm_P10.16mm_Horizontal, F.Cu at (244.7, -134.5)
- added U15: 74LS154, Package_DIP:DIP-24_W7.62mm, F.Cu at (51.4, -134.5)
- added U16: 74LS04, Package_DIP:DIP-14_W7.62mm, F.Cu at (62.3, -134.5)
- added U17: 74LS04, Package_DIP:DIP-14_W7.62mm, F.Cu at (73.1, -134.5)
- added U18: HDSP-A401, Display_7Segment:HDSP-A401, F.Cu at (62.8, -114.9)
- added U19: 74LS154, Package_DIP:DIP-24_W7.62mm, F.Cu at (51.4, -87.9)
- added U20: 74LS04, Package_DIP:DIP-14_W7.62mm, F.Cu at (73.1, -87.9)
- added U21: 74LS04, Package_DIP:DIP-14_W7.62mm, F.Cu at (62.3, -87.9)
- added U22: HDSP-A401, Display_7Segment:HDSP-A401, F.Cu at (62.8, -68.4)
- added U23: 74LS154, Package_DIP:DIP-24_W7.62mm, F.Cu at (131.8, -134.5)
- added U24: 74LS04, Package_DIP:DIP-14_W7.62mm, F.Cu at (142.7, -134.5)
- added U25: 74LS04, Package_DIP:DIP-14_W7.62mm, F.Cu at (153.5, -134.5)
- added U26: HDSP-A401, Display_7Segment:HDSP-A401, F.Cu at (143.2, -114.9)
- added U27: 74LS154, Package_DIP:DIP-24_W7.62mm, F.Cu at (131.8, -87.9)
- added U28: 74LS04, Package_DIP:DIP-14_W7.62mm, F.Cu at (142.7, -87.9)
- added U29: 74LS04, Package_DIP:DIP-14_W7.62mm, F.Cu at (153.5, -87.9)
- added U30: HDSP-A401, Display_7Segment:HDSP-A401, F.Cu at (143.2, -68.4)
- added U31: 74LS154, Package_DIP:DIP-24_W7.62mm, F.Cu at (212.2, -134.5)
- added U32: 74LS04, Package_DIP:DIP-14_W7.62mm, F.Cu at (233.9, -134.5)
- added U33: 74LS04, Package_DIP:DIP-14_W7.62mm, F.Cu at (223.0, -134.5)
- added U34: HDSP-A401, Display_7Segment:HDSP-A401, F.Cu at (223.6, -114.9)
- D100, D101, D102, D103, D104, D105, D106, D107, D108, D109, D32, D33, D34, D35, D36, D37, D38, D39, D40, D41, D42, D43, D44, D45, D46, D47, D48, D49, D50, D51, D52, D53, D54, D55, D56, D57, D58, D59, D60, D61, D62, D63, D64, D65, D66, D67, D68, D69, D70, D71, D72, D73, D74, D75, D76, D77, D78, D79, D80, D81, D82, D83, D84, D85, D86, D87, D88, D89, D90, D91, D92, D93, D94, D95, D96, D97, D98, D99: footprint Diode_THT:D_5W_P12.70mm_Horizontal -> Diode_SMD:D_SOD-123
Connections:
- U11 pad 20: /Hex to 7-Segment Decoder/A3 -> /Data_7
- U11 pad 21: /Hex to 7-Segment Decoder/A2 -> /Data_6
- U11 pad 22: /Hex to 7-Segment Decoder/A1 -> /Data_5
- U11 pad 23: /Hex to 7-Segment Decoder/A0 -> /Data_4
