File: Board_Layouts/Front_Panel/Hex_to_7-Segment_Decoder.sch (KiCad schematic (older format))
At the start: 89 parts, among them U11 74LS154, U12 74LS04, U13 74LS04, U14 HDSP-A401

Commit message: Added hex decoders to front panel
Parts:
- D100, D101, D102, D103, D104, D105, D106, D107, D108, D109, D32, D33, D34, D35, D36, D37, D38, D39, D40, D41, D42, D43, D44, D45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: footprint Diode_THT:D_5W_P12.70mm_Horizontal -> Diode_SMD:D_SOD-123
