File: Board_Layouts/CGA_Terminal/CGA_Terminal.sch (KiCad schematic (older format))
At the start: 5 parts, among them J1 Conn_01x04, J2 Conn_01x03, J3 DB9_Female_MountingHoles, U1 P8X32A-D40, U2 LM1117-3.3

Commit message: Working on CGA terminal
Parts:
- added C1, C2: 47p, symbol Device:C
- added C3: 100n, symbol Device:C
- added D1, D2: LED, symbol Device:LED
- added J1: USB_B, symbol Connector:USB_B
- added J2, J3: 8P8C, symbol Connector:8P8C
- added Q1, Q2, Q3, Q4, Q5, Q6: Q_NPN_EBC, symbol Device:Q_NPN_EBC
- added R1: 4k7, symbol Device:R
- added R10, R3, R5, R8: 600, symbol Device:R
- added R11, R13: 2k, symbol Device:R
- added R12, R14: 270, symbol Device:R
- added R15, R2: 10k, symbol Device:R
- added R16, R17, R18, R19, R20, R21: 5k6, symbol Device:R
- added R4, R9: 120, symbol Device:R
- added R6, R7: 27, symbol Device:R
- added U1: PCA9615, TSSOP10, symbol Custom_Parts:PCA9615
- added U2: FT230XS, Package_SO:SSOP-16_3.9x4.9mm_P0.635mm, symbol Interface_USB:FT230XS
- added U4: 24LC256, symbol Memory_EEPROM:24LC256
- added Y1: 14.31818 MHz, Crystal:Crystal_HC49-U_Horizontal, symbol Device:Crystal
- renumbered J1 to J4, J2 to J5, J3 to J6, U1 to U3, U2 to U5
Connections:
- net +3V3: now also C3.1, D1.2 (A), D2.2 (A), R11.1, R13.1, R15.1, U1.1 (Vdd(a)), U2.10 (3V3OUT), U2.11 (~RESET), U2.12 (VCC), U2.3 (VCCIO), U4.8 (VCC)
- net +5V: now also R3.1, R8.1, U1.10 (Vdd(b))
- net Blue: now also R18.2; no longer J6.5
- net GND: now also U3.10 (~BOE), C1.2, C2.2, C3.2, J1.4 (GND), Q1.1 (E), Q2.1 (E), Q3.1 (E), Q4.1 (E), Q5.1 (E), Q6.1 (E), R10.2, R2.2, R5.2, U1.5 (Vss), U2.13 (GND), U2.5 (GND), U4.1 (A0), U4.2 (A1), U4.3 (A2), U4.4 (GND), U4.7 (WP)
- net Green: now also R17.2; no longer J6.4
- net HSync: now also R20.2; no longer J6.8
- net Intensity: now also R19.2; no longer J6.6
- net Red: now also R16.2; no longer J6.3
- net VSync: now also R21.2; no longer J6.9
- net at U3.1 (P0): now also R11.2, U1.2 (SDA)
- net at U3.2 (P1): now also R13.2, U1.4 (SCL)
- net at U3.30 (XI): now also Y1.1
- net at U3.31 (XO): now also Y1.2
- net at U3.37 (P28): now also U4.6 (SCL)
- net at U3.38 (P29): now also R15.2, U4.5 (SDA)
- net at U3.5 (P4): now also U2.1 (TXD)
- net at U3.6 (P5): now also U2.4 (RXD)
- net at U3.7 (P6): now also U2.2 (~RTS)
- net at U3.8 (P7): now also U2.6 (~CTS)
- new net: J6.3, Q1.3 (C)
- new net: J6.4, Q2.3 (C)
- new net: J6.5, Q3.3 (C)
- new net: J6.6, Q4.3 (C)
- new net: J6.8, Q5.3 (C)
- new net: J6.9, Q6.3 (C)
- new net: Q6.2 (B), R21.1
- new net: Q5.2 (B), R20.1
- new net: Q4.2 (B), R19.1
- new net: Q3.2 (B), R18.1
- new net: Q2.2 (B), R17.1
- new net: Q1.2 (B), R16.1
- new net: R12.1, U2.14 (CBUS1)
- new net: R1.2, R2.1, U2.16 (CBUS3)
- new net: R14.1, U2.7 (CBUS2)
- new net: R7.1, U2.8 (USBDP)
- new net: R6.1, U2.9 (USBDM)
- new net: J2.7, J3.7, R10.1, R9.2, U1.6 (DSCLM)
- new net: J2.8, J3.8, R8.2, R9.1, U1.7 (DSCLP)
- new net: J2.2, J3.2, R3.2, R4.1, U1.8 (DSDAP)
- new net: J2.1, J3.1, R4.2, R5.1, U1.9 (DSDAM)
- new net: C1.1, J1.3 (D+), R7.2
- new net: C2.1, J1.2 (D-), R6.2
- new net: D1.1 (K), R12.2
- new net: D2.1 (K), R14.2
- new net: J1.1 (VBUS), R1.1
- no-connect marks 3 -> 28
Other:
- moved on the sheet: J4, U3
